File: AB201.kicad_pcb (KiCad board)
At the start: 2 copper layers, 200 x 100 mm, 90 parts, among them J1 CONN_01X08, J10 screwhole, J2 CONN_01X04, J3 CONN_01X08, J4 HEATSINK, J5 screwhole, J6 screwhole, J7 screwhole, J8 screwhole, J9 screwhole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

Commit message: PCB layout updated
Parts:
- moved D4 1.58 mm to (200.0, 45.5), turned to 0 degrees
Routing:
- net Net-(D4-Pad2): track 188.6 -> 194.3 mm
- net Net-(D4-Pad1): track 198.2 -> 193.2 mm
Other:
- board text added: "HAOS REDRO PN: 0000 0002 www.haosredro.com Licensed under CERN OHL v1.2 or later"
- board text removed: "HAOS REDRO AB201 www.haosredro.com"
- board text removed: "Licensed under CERN OHL v.1.2 or later"
Changed lines of the file:
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@@
     (area 47.964286 26.225 252.035714 130.775)
     (thickness 1.6)
-    (drawings 30)
-    (tracks 460)
+    (drawings 29)
+    (tracks 462)
     (zones 0)
     (modules 90)
@@
   )
   (setup
-    (last_trace_width 0.5)
+    (last_trace_width 1)
     (user_trace_width 0.5)
     (user_trace_width 1)
@@
   )
   (module Diodes_SMD:D_SMA (layer F.Cu)
-    (at 201.5 45 180)
+    (at 200 45.5)
     (descr "Diode SMA (DO-214AC)")
     (tags "Diode SMA (DO-214AC)")
     (attr smd)
-    (fp_text reference D4 (at -5 0 180) (layer F.SilkS)
+    (fp_text reference D4 (at -5 0) (layer F.SilkS)
       (effects (font (size 1 1) (thickness 0.15)))
     )
-    (fp_text value 4001 (at 0 2.6 180) (layer F.Fab)
+    (fp_text value 4001 (at 0 2.6) (layer F.Fab)
       (effects (font (size 1 1) (thickness 0.15)))
     )
-    (fp_text user %R (at 0 -2.5 180) (layer F.Fab)
+    (fp_text user %R (at 0 -2.5) (layer F.Fab)
       (effects (font (size 1 1) (thickness 0.15)))
     )
@@
     (fp_line (start -3.4 1.65) (end 2 1.65) (layer F.SilkS) (width 0.12))
     (fp_line (start -3.4 -1.65) (end 2 -1.65) (layer F.SilkS) (width 0.12))
-    (pad 1 smd rect (at -2 0 180) (size 2.5 1.8) (layers F.Cu F.Paste F.Mask)
+    (pad 1 smd rect (at -2 0) (size 2.5 1.8) (layers F.Cu F.Paste F.Mask)
       (net 13 "Net-(D4-Pad1)"))
-    (pad 2 smd rect (at 2 0 180) (size 2.5 1.8) (layers F.Cu F.Paste F.Mask)
+    (pad 2 smd rect (at 2 0) (size 2.5 1.8) (layers F.Cu F.Paste F.Mask)
       (net 14 "Net-(D4-Pad2)"))
     (model ${KISYS3DMOD}/Diodes_SMD.3dshapes/D_SMA.wrl
@@
       (net 30 "Net-(L1-Pad2)"))
   )
-  (gr_text "Licensed under CERN\nOHL v.1.2 or later" (at 213 113) (layer F.SilkS)
-    (effects (font (size 1.5 1.5) (thickness 0.3)))
-  )
-  (gr_text "HAOS REDRO AB201\nwww.haosredro.com" (at 235 104.5) (layer F.SilkS)
-    (effects (font (size 1.5 1.5) (thickness 0.3)))
+  (gr_text "HAOS REDRO PN: 0000 0002\nwww.haosredro.com\nLicensed under CERN OHL v1.2 or later" (at 180.5 90) (layer B.Cu)
+    (effects (font (size 1.5 1.5) (thickness 0.3)) (justify mirror))
   )
   (gr_line (start 120.5 42.5) (end 121.5 41.5) (angle 90) (layer F.SilkS) (width 0.2))
@@
   (segment (start 70.05 106.7) (end 70 106.75) (width 0.5) (layer F.Cu) (net 11))
   (segment (start 62.58 104) (end 67.5 104) (width 0.5) (layer F.Cu) (net 12))
-  (segment (start 94 67.5) (end 68.5 67.5) (width 1) (layer F.Cu) (net 13))
-  (segment (start 195.75 67.25) (end 195.5 67.5) (width 1) (layer F.Cu) (net 13))
-  (via (at 195.5 67.5) (size 1) (drill 0.6) (layers F.Cu B.Cu) (net 13))
-  (segment (start 195.5 67.5) (end 179.5 67.5) (width 1) (layer B.Cu) (net 13))
-  (via (at 179.5 67.5) (size 1) (drill 0.6) (layers F.Cu B.Cu) (net 13))
-  (segment (start 179.5 67.5) (end 130 67.5) (width 1) (layer F.Cu) (net 13))
-  (via (at 130 67.5) (size 1) (drill 0.6) (layers F.Cu B.Cu) (net 13))
-  (segment (start 130 67.5) (end 94 67.5) (width 1) (layer B.Cu) (net 13))
-  (via (at 94 67.5) (size 1) (drill 0.6) (layers F.Cu B.Cu) (net 13))
-  (segment (start 195.75 52) (end 195.75 67.25) (width 1) (layer F.Cu) (net 13))
-  (segment (start 61.08 46.58) (end 57.54 46.58) (width 1) (layer B.Cu) (net 13))
-  (segment (start 62 47.5) (end 61.08 46.58) (width 1) (layer B.Cu) (net 13))
-  (segment (start 62 51.5) (end 62 47.5) (width 1) (layer B.Cu) (net 13))
-  (via (at 62 51.5) (size 1) (drill 0.6) (layers F.Cu B.Cu) (net 13))
-  (segment (start 62 61) (end 62 51.5) (width 1) (layer F.Cu) (net 13))
+  (segment (start 195.5 67.5) (end 195.5 55.5) (width 1) (layer F.Cu) (net 13))
   (segment (start 68.5 67.5) (end 62 61) (width 1) (layer F.Cu) (net 13))
-  (segment (start 195.75 52) (end 197.5 52) (width 1) (layer F.Cu) (net 13))
-  (segment (start 201.5 47) (end 203.5 45) (width 1) (layer F.Cu) (net 13))
-  (segment (start 201.5 48) (end 201.5 47) (width 1) (layer F.Cu) (net 13))
-  (segment (start 197.5 52) (end 201.5 48) (width 1) (layer F.Cu) (net 13))
-  (segment (start 199.5 31.75) (end 202.75 31.75) (width 1) (layer F.Cu) (net 13))
-  (segment (start 203.5 32.5) (end 203.5 45) (width 1) (layer F.Cu) (net 13))
-  (segment (start 202.75 31.75) (end 203.5 32.5) (width 1) (layer F.Cu) (net 13))
-  (segment (start 94 71.5) (end 67.5 71.5) (width 1) (layer F.Cu) (net 14))
-  (segment (start 193.5 50.5) (end 193.5 71.5) (width 1) (layer F.Cu) (net 14))
-  (via (at 193.5 71.5) (size 1) (drill 0.6) (layers F.Cu B.Cu) (net 14))
-  (segment (start 193.5 71.5) (end 179.5 71.5) (width 1) (layer B.Cu) (net 14))
+  (segment (start 62 61) (end 62 51.5) (width 1) (layer F.Cu) (net 13))
+  (via (at 62 51.5) (size 1) (drill 0.6) (layers F.Cu B.Cu) (net 13))
+  (segment (start 62 51.5) (end 62 47.5) (width 1) (layer B.Cu) (net 13))
+  (segment (start 62 47.5) (end 61.08 46.58) (width 1) (layer B.Cu) (net 13))
+  (segment (start 57.54 46.58) (end 61.08 46.58) (width 1) (layer B.Cu) (net 13))
+  (via (at 94 67.5) (size 1) (drill 0.6) (layers F.Cu B.Cu) (net 13))
+  (segment (start 130 67.5) (end 94 67.5) (width 1) (layer B.Cu) (net 13))
+  (via (at 130 67.5) (size 1) (drill 0.6) (layers F.Cu B.Cu) (net 13))
+  (segment (start 179.5 67.5) (end 130 67.5) (width 1) (layer F.Cu) (net 13))
+  (via (at 179.5 67.5) (size 1) (drill 0.6) (layers F.Cu B.Cu) (net 13))
+  (segment (start 195.5 67.5) (end 179.5 67.5) (width 1) (layer B.Cu) (net 13))
+  (via (at 195.5 67.5) (size 1) (drill 0.6) (layers F.Cu B.Cu) (net 13))
+  (segment (start 94 67.5) (end 68.5 67.5) (width 1) (layer F.Cu) (net 13))
+  (segment (start 195.75 55.25) (end 195.75 52) (width 1) (layer F.Cu) (net 13))
+  (segment (start 195.5 55.5) (end 195.75 55.25) (width 1) (layer F.Cu) (net 13))
+  (segment (start 198 45.5) (end 198 43.5) (width 1) (layer F.Cu) (net 13))
+  (segment (start 196.5 34.75) (end 199.5 31.75) (width 1) (layer F.Cu) (net 13))
+  (segment (start 196.5 42) (end 196.5 34.75) (width 1) (layer F.Cu) (net 13))
+  (segment (start 198 43.5) (end 196.5 42) (width 1) (layer F.Cu) (net 13))
+  (segment (start 195.75 52) (end 195.75 47.75) (width 1) (layer F.Cu) (net 13))
+  (segment (start 195.75 47.75) (end 198 45.5) (width 1) (layer F.Cu) (net 13))
+  (segment (start 199.5 39.25) (end 199.75 39.25) (width 1) (layer F.Cu) (net 14) (status C00000))
+  (segment (start 199.75 39.25) (end 202 41.5) (width 1) (layer F.Cu) (net 14) (status 400000))
+  (segment (start 202 41.5) (end 202 45.5) (width 1) (layer F.Cu) (net 14) (status 800000))
+  (segment (start 200 71.5) (end 200 49.5) (width 1) (layer F.Cu) (net 14))
+  (via (at 200 71.5) (size 1) (drill 0.6) (layers F.Cu B.Cu) (net 14))
+  (segment (start 200 71.5) (end 179.5 71.5) (width 1) (layer B.Cu) (net 14))
   (via (at 179.5 71.5) (size 1) (drill 0.6) (layers F.Cu B.Cu) (net 14))
   (segment (start 179.5 71.5) (end 130 71.5) (width 1) (layer F.Cu) (net 14))
@@
   (segment (start 130 71.5) (end 94 71.5) (width 1) (layer B.Cu) (net 14))
   (via (at 94 71.5) (size 1) (drill 0.6) (layers F.Cu B.Cu) (net 14))
-  (segment (start 199 45) (end 193.5 50.5) (width 1) (layer F.Cu) (net 14))
-  (segment (start 55 59) (end 55 49.12) (width 1) (layer F.Cu) (net 14))
+  (segment (start 55 49.12) (end 55 59) (width 1) (layer F.Cu) (net 14))
   (segment (start 67.5 71.5) (end 55 59) (width 1) (layer F.Cu) (net 14))
-  (segment (start 199.5 45) (end 199 45) (width 1) (layer F.Cu) (net 14))
-  (segment (start 199.5 39.25) (end 199.5 45) (width 1) (layer F.Cu) (net 14))
+  (segment (start 94 71.5) (end 67.5 71.5) (width 1) (layer F.Cu) (net 14))
+  (segment (start 202 47.5) (end 202 45.5) (width 1) (layer F.Cu) (net 14) (status 800000))
+  (segment (start 200 49.5) (end 202 47.5) (width 1) (layer F.Cu) (net 14))
   (segment (start 64.5 44.04) (end 65.54 44.04) (width 0.5) (layer F.Cu) (net 15))
   (segment (start 72 51.5) (end 76.25 51.5) (width 0.5) (layer F.Cu) (net 15))
@@
   (segment (start 196 117) (end 204.6 108.4) (width 3) (layer B.Cu) (net 43))
   (segment (start 189.5 39) (end 189.5 42.5) (width 3) (layer B.Cu) (net 44))
-  (segment (start 189.5 42.5) (end 192.5 45.5) (width 3) (layer B.Cu) (net 44))
-  (segment (start 192.5 45.5) (end 214 45.5) (width 3) (layer B.Cu) (net 44))
-  (segment (start 214 45.5) (end 215.4 46.9) (width 3) (layer B.Cu) (net 44))
   (segment (start 215.4 46.9) (end 215.4 52) (width 3) (layer B.Cu) (net 44))
+  (segment (start 214 45.5) (end 215.4 46.9) (width 3) (layer B.Cu) (net 44))
+  (segment (start 192.5 45.5) (end 214 45.5) (width 3) (layer B.Cu) (net 44))
+  (segment (start 189.5 42.5) (end 192.5 45.5) (width 3) (layer B.Cu) (net 44))
   (segment (start 127.5 47.55) (end 127.5 45.5) (width 0.5) (layer F.Cu) (net 45))
   (segment (start 128.5 44.5) (end 137 44.5) (width 0.5) (layer F.Cu) (net 45))
@@
   (segment (start 179.5 69.5) (end 130 69.5) (width 0.5) (layer F.Cu) (net 51))
   (via (at 179.5 69.5) (size 0.6) (drill 0.4) (layers F.Cu B.Cu) (net 51))
-  (segment (start 195.5 69.5) (end 179.5 69.5) (width 0.5) (layer B.Cu) (net 51))
-  (via (at 195.5 69.5) (size 0.6) (drill 0.4) (layers F.Cu B.Cu) (net 51))
-  (segment (start 205.5 69.5) (end 195.5 69.5) (width 0.5) (layer F.Cu) (net 51))
+  (segment (start 202 69.5) (end 179.5 69.5) (width 0.5) (layer B.Cu) (net 51))
+  (via (at 202 69.5) (size 0.6) (drill 0.4) (layers F.Cu B.Cu) (net 51))
+  (segment (start 205.5 69.5) (end 202 69.5) (width 0.5) (layer F.Cu) (net 51))
   (segment (start 223.38 51.62) (end 205.5 69.5) (width 0.5) (layer F.Cu) (net 51))
   (segment (start 226 81) (end 227.5 81) (width 0.5) (layer F.Cu) (net 51))
@@
       (pts
         (xy 250 48) (xy 250 40) (xy 230.5 40) (xy 227.5 43) (xy 221.5 43)
-        (xy 221.5 28) (xy 214.5 28) (xy 214.5 47.5) (xy 217.5 50) (xy 234 50)
+        (xy 221.5 28) (xy 214.5 28) (xy 214.5 47) (xy 217.5 50) (xy 234 50)
         (xy 236 48)
       )

Commit message: PCB changes
Parts:
- moved R12 3.50 mm to (95.5, 112.0)
Routing:
- net /OUT: track 485.5 -> 136.6 mm, vias 20 -> 34
- net Net-(Q11-Pad1): track 149.0 -> 200.5 mm, vias 1 -> 4
- net Net-(Q10-Pad2): track 162.5 -> 187.2 mm, vias 1 -> 4
- net Net-(J1-Pad8): track 156.4 -> 169.0 mm, vias 3 -> 2
- net Net-(D4-Pad1): track 193.2 -> 202.5 mm, vias 5 -> 3
- net Net-(D4-Pad2): track 194.3 -> 201.6 mm, vias 4 -> 2
- net Net-(F1-Pad1): track 6.25 -> 0.00 mm
- net Net-(C16-Pad1): track 92.7 -> 91.0 mm, vias 0 -> 2
- net /V+: track 101.7 -> 102.1 mm, vias 2 -> 4
