File: AB201.sch (KiCad schematic (older format))
At the start: 90 parts, among them J1 CONN_01X08, J10 screwhole, J2 CONN_01X04, J3 CONN_01X08, J4 HEATSINK, J5 screwhole, J6 screwhole, J7 screwhole, J8 screwhole, J9 screwhole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

Commit message: PCB changes
Parts:
- C1, C10, C11, C13, C14, C15, C16, C17, C18, C2, C29, C3, C4, C5, C6, C7, C8, C9: symbol C -> AB201-rescue:C
- C12, C19, C20, C21, C22, C23, C24, C25, C26, C27, C28: symbol CP -> AB201-rescue:CP
- D1: symbol LED -> AB201-rescue:LED
- D2: symbol DIAC -> AB201-rescue:DIAC
- D3: symbol Q_TRIAC_AAG -> AB201-rescue:Q_TRIAC_AAG
- D4: symbol D -> AB201-rescue:D
- F1, F2: symbol Fuse -> AB201-rescue:Fuse
- J1, J3: symbol CONN_01X08 -> AB201-rescue:CONN_01X08
- J10, J5, J6, J7, J8, J9: symbol Conn_01x01 -> AB201-rescue:Conn_01x01
- J2: symbol CONN_01X04 -> AB201-rescue:CONN_01X04
- J4: symbol Conn_01x06 -> AB201-rescue:Conn_01x06
- L1: symbol L -> AB201-rescue:L
- Q1, Q3, Q5: symbol Q_NPN_BEC -> AB201-rescue:Q_NPN_BEC
- Q10, Q11, Q13, Q15, Q6: symbol Q_PNP_BCE -> AB201-rescue:Q_PNP_BCE
- Q12, Q14, Q16, Q7, Q8, Q9: symbol Q_NPN_BCE -> AB201-rescue:Q_NPN_BCE
- Q2, Q4: symbol Q_PNP_BEC -> AB201-rescue:Q_PNP_BEC
- R1, R10, R11, R12, R13, R14, R15, R16, R17, R18, R19, R2, R20, R21, R22, R23, R24, R3, R4, R5, R6, R7, R8, R9: symbol R -> AB201-rescue:R
- RE1: symbol RELAY_OMRON_G2R_1A_E -> AB201-rescue:RELAY_OMRON_G2R_1A_E-HR-PARTS
- RV1: symbol POT -> AB201-rescue:POT
- SW1: symbol THERMOSTAT_NC -> AB201-rescue:THERMOSTAT_NC-HR-PARTS
- TH1: symbol Thermistor -> AB201-rescue:Thermistor
